File: Differential_Probe_PCB/Differential_Probe.kicad_pcb (KiCad board)
At the start: 4 copper layers, 100 x 50 mm, 158 parts, among them IC101 AD8130ARM, J101 Conn_01x01_Socket, J102 Conn_Coaxial, J103 Conn_01x01_Socket, J104 USB_C_Receptacle_PowerOnly_6P, K101 EE2-5NU, K102 EE2-5NU, SW101 SW_SPDT, SW102 SW_SPDT, U101 TPS7A39, U102 TPS65130RGE, U103 THS3491xDDA, U106 LM321

Commit message: .
Parts:
- added C159: 10u, Capacitor_SMD:C_1206_3216Metric, B.Cu at (131.2, 141.8)
- added C163: 330n, Capacitor_SMD:C_1206_3216Metric, B.Cu at (127.0, 139.8)
- added C164: 100n, Capacitor_SMD:C_0603_1608Metric, B.Cu at (131.2, 139.8)
- added C165: 10u, Capacitor_SMD:C_1206_3216Metric, B.Cu at (136.0, 141.8)
- added C166: 100n, Capacitor_SMD:C_0603_1608Metric, B.Cu at (136.0, 139.8)
- added D111: RLED, Diode_SMD:D_1206_3216Metric, F.Cu at (119.5, 145.1)
- added GND: TestPoint, TestPoint:TestPoint_THTPad_D1.0mm_Drill0.5mm, F.Cu at (132.8, 118.8)
- added GND: TestPoint, TestPoint:TestPoint_THTPad_D1.0mm_Drill0.5mm, F.Cu at (129.4, 131.6)
- added GND: TestPoint, TestPoint:TestPoint_THTPad_D1.0mm_Drill0.5mm, F.Cu at (146.5, 132.5)
- added GND: TestPoint, TestPoint:TestPoint_THTPad_D1.0mm_Drill0.5mm, F.Cu at (145.5, 125.0)
- added GND: TestPoint, TestPoint:TestPoint_THTPad_D1.0mm_Drill0.5mm, F.Cu at (110.2, 106.0)
- added Q101: AO3401A, Package_TO_SOT_SMD:SOT-23, B.Cu at (124.0, 143.8)
- added Q102: AO3400A, Package_TO_SOT_SMD:SOT-23, B.Cu at (120.2, 140.0)
- added R140: 1k, Resistor_SMD:R_0603_1608Metric, B.Cu at (119.5, 145.1)
- added R155: 10k, Resistor_SMD:R_0603_1608Metric, B.Cu at (124.0, 148.0)
- added R159: 49.9R, Resistor_SMD:R_1206_3216Metric, F.Cu at (141.8, 138.0)
- added R160: 10k, Resistor_SMD:R_0603_1608Metric, B.Cu at (117.5, 140.0)
- added R161: 10R, Resistor_SMD:R_0603_1608Metric, B.Cu at (116.0, 140.0)
- added R162: 10R, Resistor_SMD:R_0603_1608Metric, B.Cu at (123.5, 139.8)
- added R163: 3.3M, Resistor_SMD:R_0603_1608Metric, B.Cu at (125.0, 139.8)
- added R164: 100k, Resistor_SMD:R_0603_1608Metric, B.Cu at (128.0, 147.0)
- added R165: 1k, Resistor_SMD:R_0603_1608Metric, B.Cu at (126.5, 147.0)
- added R166: 10R, Resistor_SMD:R_0603_1608Metric, B.Cu at (124.0, 146.5)
- added R167: 10k, Resistor_SMD:R_0603_1608Metric, F.Cu at (136.0, 145.2)
- added R168: 2k, Resistor_SMD:R_0603_1608Metric, F.Cu at (136.0, 146.8)
- added R169: 10k, Resistor_SMD:R_0603_1608Metric, F.Cu at (145.8, 137.0)
- added R170: 10k, Resistor_SMD:R_0603_1608Metric, F.Cu at (147.2, 137.0)
- added R171: 2k, Resistor_SMD:R_0603_1608Metric, F.Cu at (136.0, 142.2)
- added R172: 10k, Resistor_SMD:R_0603_1608Metric, F.Cu at (136.0, 143.8)
- added TP103: TestPoint, TestPoint:TestPoint_THTPad_D1.0mm_Drill0.5mm, F.Cu at (145.5, 123.0)
- added TP104: TestPoint, TestPoint:TestPoint_THTPad_D1.0mm_Drill0.5mm, F.Cu at (145.5, 127.0)
- added TP105: TestPoint, TestPoint:TestPoint_THTPad_D1.0mm_Drill0.5mm, F.Cu at (146.5, 134.5)
- added TP106: TestPoint, TestPoint:TestPoint_THTPad_D1.0mm_Drill0.5mm, F.Cu at (128.8, 140.2)
- added TP107: TestPoint, TestPoint:TestPoint_THTPad_D1.0mm_Drill0.5mm, F.Cu at (144.8, 139.5)
- added TP108: TestPoint, TestPoint:TestPoint_THTPad_D1.0mm_Drill0.5mm, F.Cu at (110.2, 108.5)
- added TP109: TestPoint, TestPoint:TestPoint_THTPad_D1.0mm_Drill0.5mm, F.Cu at (134.8, 118.8)
- added TP110: TestPoint, TestPoint:TestPoint_THTPad_D1.0mm_Drill0.5mm, F.Cu at (146.5, 130.5)
- added TP111: TestPoint, TestPoint:TestPoint_THTPad_D1.0mm_Drill0.5mm, F.Cu at (129.5, 129.0)
- added U104: LM339, Package_SO:TSSOP-14_4.4x5mm_P0.65mm, B.Cu at (133.2, 146.0)
- C101, C110: value C_Small -> 120p
- C102, C111, C121, C125: value C_Small -> 50p
- C103, C112: value C_Small -> 20p
- C104, C113, C122, C126: value C_Trim_Small -> 10p
- C105, C106, C107, C108, C109, C114, C115, C116, C117, C118: value C_Small -> 10p
- C119, C123: value C_Small -> 1.5n
- C120, C124: value C_Small -> 510p
- J102: footprint Connector_Coaxial:BNC_Amphenol_031-6575_Horizontal -> SamacSys_Parts:2269901
- J104: footprint Connector_USB:USB_C_Receptacle_HRO_TYPE-C-31-M-17 -> Connector_USB:USB_C_Receptacle_GCT_USB4125-xx-x_6P_TopMnt_Horizontal
- R103, R111: value 184k -> 68k
- R119, R126: value 22k, 0.1% -> 5.1k, 0.1%
- R157, R158: moved to B.Cu
- moved R157 16.8 mm to (147.0, 141.6)
- moved R158 16.7 mm to (142.5, 141.6)
- moved R142 13.4 mm to (142.0, 140.0)
- moved R124 11.4 mm to (158.0, 123.4), turned to -90 degrees
- moved R121 11.4 mm to (158.0, 126.5), turned to -90 degrees
- moved R122 11.0 mm to (169.0, 126.6)
- moved R125 11.0 mm to (169.0, 123.4)
- moved R148 7.50 mm to (142.5, 140.0)
- moved RV103 6.05 mm to (147.3, 143.5)
- moved C155 5.84 mm to (147.6, 146.8), turned to 90 degrees
- moved C160 5.84 mm to (149.6, 146.8), turned to 90 degrees
- moved U106 5.84 mm to (145.0, 146.8)
- moved C157 5.84 mm to (140.3, 146.8)
- moved C158 5.84 mm to (142.3, 146.8)
- moved R150 5.10 mm to (147.0, 140.0)
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Connections:
- net /Input_attenuator/x10_attentuation renamed /Buttons_indication/x10_attenuation
- net Att_P renamed /Amplifier/Att_P
- net Net-(IC101-OUT) renamed /Amplifier/Single_ended_input
Routing:
- net -12V: track 20.7 -> 76.9 mm, vias 12 -> 16
- net +12V: track 22.2 -> 58.3 mm, vias 14 -> 18
- net GND: track 97.3 -> 131.6 mm, vias 60 -> 120
- net /Amplifier/BW_Limit: track 21.1 -> 49.1 mm
- net Net-(D111-K): track 0.00 -> 23.0 mm, vias 0 -> 1
- net /Buttons_indication/x10_attenuation: track 33.7 -> 54.8 mm
- net Net-(R155-Pad2): track 0.00 -> 20.7 mm
- net Net-(U104A--): track 0.00 -> 20.4 mm, vias 0 -> 1
- net Net-(U104B-+): track 0.00 -> 17.6 mm, vias 0 -> 1
- net +5V: track 0.00 -> 14.6 mm, vias 0 -> 18
- net Net-(U104C-+): track 0.00 -> 13.0 mm
- net /Amplifier/Att_N: track 40.4 -> 51.1 mm
- net Net-(Q101-S): track 0.00 -> 9.96 mm
- net /Amplifier/Att_P: track 40.4 -> 49.4 mm
- net Net-(U106--): track 2.28 -> 11.0 mm
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- added copper zone on In2.Cu, net +12V
- added copper zone on In2.Cu, net +5V
- added copper zone on In2.Cu, net -12V
Other:
- outline, holes or cut-outs redrawn
- board text added: "+"
- board text added: "-"
- board text added: "HV_Differential_Probe v1.0"
- board text added: "Offset adj"
- board text added: "x10 adj"
- board text added: "x100 adj"

Commit message: After 1st debug update to sch
Parts:
- C101, C110: value 120p -> 120p, 1%
- C102, C111: value 50p -> 50p, 1%
- C103, C112: value 20p -> 10p, 1%
- C104, C113, C122, C126: value 10p -> 8-30p
- C119, C123: value 1.5n -> 1.5n, 1%
- C120, C124: value 510p -> 420pF, 1%
- C121, C125: value 50p -> 20pF, 1%/50pF 1%
- C139: value xxx -> 6.8p
- C142: value 220n -> 6.8p
- C146: value xxx -> 10n
- C147: value xxx -> 4.7n
- R103, R111: value 68k -> 62k, 0.1%
- R104, R110: value 0R -> 1.5k, 0.1%
- R130: value 90.9k -> 100k
- R131: value xxx -> 1M
- R132: value xxx -> 88k
- R133: value xxx -> 100k
- R135: value xxx -> 1.3M
- R157, R158: value 100k -> 10k
- R167, R172: value 10k -> 2.2k
- R168, R171: value 2k -> 10k
- RV101: value 500R -> 1k
- RV102: value 220R -> 100R
- SW101, SW102: value SW_SPDT -> TL2202EEYA
- U106: value LM321 -> OPA187I
Changed lines of the file:
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@@
 			)
 		)
-		(property "Value" "10k"
+		(property "Value" "2.2k"
 			(at 0 1.43 0)
 			(layer "F.Fab")
@@
 			)
 		)
-		(property "Value" "120p"
+		(property "Value" "120p, 1%"
 			(at 0 1.43 90)
 			(layer "F.Fab")
@@
 			)
 		)
-		(property "Value" "510p"
+		(property "Value" "420pF, 1%"
 			(at 0 1.43 90)
 			(layer "F.Fab")
@@
 			)
 		)
-		(property "Value" "20p"
+		(property "Value" "10p, 1%"
 			(at 0 1.43 90)
 			(layer "F.Fab")
@@
 			)
 		)
-		(property "Value" "1.5n"
+		(property "Value" "1.5n, 1%"
 			(at 0 1.43 90)
 			(layer "F.Fab")
@@
 			)
 		)
-		(property "Value" "SW_SPDT"
+		(property "Value" "TL2202EEYA"
 			(at 2.5 -3 0)
 			(layer "F.SilkS")
@@
 			)
 		)
-		(property "Value" "xxx"
+		(property "Value" "100k"
 			(at 0 1.43 90)
 			(layer "F.Fab")
@@
 			)
 		)
-		(property "Value" "500R"
+		(property "Value" "1k"
 			(at -2.54 3.67 90)
 			(layer "F.Fab")
@@
 			)
 		)
-		(property "Value" "2k"
+		(property "Value" "10k"
 			(at 0 1.43 0)
 			(layer "F.Fab")
@@
 			)
 		)
-		(property "Value" "1.5n"
+		(property "Value" "1.5n, 1%"
 			(at 0 1.43 90)
 			(layer "F.Fab")
@@
 			)
 		)
-		(property "Value" "220n"
+		(property "Value" "6.8p"
 			(at 0 1.43 90)
 			(layer "F.Fab")
@@
 			)
 		)
-		(property "Value" "10p"
+		(property "Value" "8-30p"
 			(at 0 3.25 0)
 			(layer "F.Fab")
@@
 			)
 		)
-		(property "Value" "20p"
+		(property "Value" "10p, 1%"
 			(at 0 1.43 90)
 			(layer "F.Fab")
@@
 			)
 		)
-		(property "Value" "xxx"
+		(property "Value" "88k"
 			(at 0 1.43 0)
 			(layer "F.Fab")
@@
 			)
 		)
-		(property "Value" "10p"
+		(property "Value" "8-30p"
 			(at 0 3.25 0)
 			(layer "F.Fab")
@@
 			)
 		)
-		(property "Value" "120p"
+		(property "Value" "120p, 1%"
 			(at 0 1.43 90)
 			(layer "F.Fab")
@@
 			)
 		)
-		(property "Value" "220R"
+		(property "Value" "100R"
 			(at -2.54 3.67 90)
 			(layer "F.Fab")
@@
 			)
 		)
-		(property "Value" "510p"
+		(property "Value" "420pF, 1%"
 			(at 0 1.43 90)
 			(layer "F.Fab")
@@
 			)
 		)
-		(property "Value" "0R"
+		(property "Value" "1.5k, 0.1%"
 			(at 0 1.43 0)
 			(layer "F.Fab")
@@
 			)
 		)
-		(property "Value" "xxx"
+		(property "Value" "1.3M"
 			(at 0 1.43 90)
 			(layer "F.Fab")
@@
 			)
 		)
-		(property "Value" "68k"
+		(property "Value" "62k, 0.1%"
 			(at 0 1.43 180)
 			(layer "F.Fab")
@@
 			)
 		)
-		(property "Value" "50p"
+		(property "Value" "20pF, 1%/50pF 1%"
 			(at 0 1.43 90)
 			(layer "F.Fab")
@@
 			)
 		)
-		(property "Value" "2k"
+		(property "Value" "10k"
 			(at 0 1.43 0)
 			(layer "F.Fab")
@@
 			)
 		)
-		(property "Value" "SW_SPDT"
+		(property "Value" "TL2202EEYA"
 			(at 2.5 -3 0)
 			(layer "F.SilkS")
@@
 			)
 		)
-		(property "Value" "10k"
+		(property "Value" "2.2k"
 			(at 0 1.43 0)
 			(layer "F.Fab")
@@
 			)
 		)
-		(property "Value" "10p"
+		(property "Value" "8-30p"
 			(at 0 3.25 0)
 			(layer "F.Fab")
@@
 			)
 		)
-		(property "Value" "xxx"
+		(property "Value" "1M"
 			(at 0 1.43 90)
 			(layer "F.Fab")
@@
 			)
 		)
-		(property "Value" "50p"
+		(property "Value" "50p, 1%"
 			(at 0 1.43 90)
 			(layer "F.Fab")
@@
 			)
 		)
-		(property "Value" "xxx"
+		(property "Value" "4.7n"
 			(at 0 1.43 0)
 			(layer "F.Fab")
@@
 			)
 		)
-		(property "Value" "10p"
+		(property "Value" "8-30p"
 			(at 0 3.25 0)
 			(layer "F.Fab")
@@
 			)
 		)
-		(property "Value" "xxx"
+		(property "Value" "10n"
 			(at 0 1.43 0)
 			(layer "F.Fab")
@@
 			)
 		)
-		(property "Value" "50p"
+		(property "Value" "50p, 1%"
 			(at 0 1.43 90)
 			(layer "F.Fab")
@@
 			)
 		)
-		(property "Value" "xxx"
+		(property "Value" "6.8p"
 			(at 0 1.43 90)
 			(layer "F.Fab")
@@
 			)
 		)
-		(property "Value" "68k"
+		(property "Value" "62k, 0.1%"
 			(at 0 1.43 180)
 			(layer "F.Fab")
@@
 			)
 		)
-		(property "Value" "50p"
+		(property "Value" "20pF, 1%/50pF 1%"
 			(at 0 1.43 90)
 			(layer "F.Fab")
@@
 			)
 		)
-		(property "Value" "0R"
+		(property "Value" "1.5k, 0.1%"
 			(at 0 1.43 0)
 			(layer "F.Fab")
@@
 			)
 		)
-		(property "Value" "90.9k"
+		(property "Value" "100k"
 			(at 0 -1.43 0)
 			(layer "B.Fab")
@@
 			)
 		)
-		(property "Value" "100k"
+		(property "Value" "10k"
 			(at 0 -1.43 0)
 			(layer "B.Fab")
@@
 			)
 		)
-		(property "Value" "LM321"
+		(property "Value" "OPA187I"
 			(at 0 -2.4 90)
 			(layer "B.Fab")
@@
 			)
 		)
-		(property "Value" "100k"
+		(property "Value" "10k"
 			(at 0 -1.43 180)
 			(layer "B.Fab")
