File: Differential_Probe_PCB/Amplifier.kicad_sch (KiCad schematic)
At the start: 34 parts, among them IC101 AD8130ARM, K102 EE2-5NU, U103 THS3491xDDA, U106 LM321

Commit message: .
Parts:
- added TP105, TP106, TP107: TestPoint, TestPoint:TestPoint_THTPad_D1.0mm_Drill0.5mm, symbol Connector:TestPoint
- R157, R158: value 100k -> 10k
Connections:
- net at R142.2, U106.3 (-), U106.4: now also TP107.1
- net at R136.1, R139.1, R143.2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: now also TP106.1
- net Single_ended_input: now reaches IC101.6 (OUT), R141.1, R156.2
- net Single_ended_input: now also TP105.1

Commit message: After 1st debug update to sch
Parts:
- U106: value LM321 -> OPA187I
Other:
- note added: "Fucked up pinout"
- note added: "R142 - 10k"
- note added: "R148 - 200R"
- note added: "R150 - 0R"
- note added: "changed 6.8u to 10u"
Changed lines of the file:
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@@
+		)
+	)
+	(text "R142 - 10k"
+		(exclude_from_sim no)
+		(at 146.304 101.346 0)
+		(effects
+			(font
+				(size 1.27 1.27)
+				(color 255 0 0 1)
+			)
 		)
 	)
@@
 		)
 	)
+	(text "R148 - 200R\n\n"
+		(exclude_from_sim no)
+		(at 60.96 147.828 0)
+		(effects
+			(font
+				(size 1.27 1.27)
+				(color 255 0 0 1)
+			)
+		)
+	)
 	(text "Bias current comp\n(optional)\n"
 		(exclude_from_sim no)
@@
 		)
 	)
+	(text "R150 - 0R\n\n"
+		(exclude_from_sim no)
+		(at 60.198 178.308 0)
+		(effects
+			(font
+				(size 1.27 1.27)
+				(color 255 0 0 1)
+			)
+		)
+	)
 	(text "Input offset correction"
 		(exclude_from_sim no)
@@
 				(thickness 0.5)
 				(bold yes)
+			)
+		)
+	)
+	(text "Fucked up pinout"
+		(exclude_from_sim no)
+		(at 139.7 172.466 0)
+		(effects
+			(font
+				(size 1.27 1.27)
+				(color 255 0 0 1)
+			)
+		)
+	)
+	(text "changed 6.8u to 10u\n"
+		(exclude_from_sim no)
+		(at 166.878 39.116 0)
+		(effects
+			(font
+				(size 1.27 1.27)
+				(color 255 0 0 1)
 			)
 		)
@@
 			)
 		)
-		(property "Value" "LM321"
+		(property "Value" "OPA187I"
 			(at 132.334 161.8294 0)
 			(effects

Commit message: .
Other:
- note added: "C150, C153 - 10u"
- note added: "Wrong pinout of U106"
- note added: "~550mV"
- note removed: "Fucked up pinout"
- note removed: "changed 6.8u to 10u"
Changed lines of the file:
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@@
+		)
+	)
+	(text "~550mV"
+		(exclude_from_sim no)
+		(at 147.828 134.62 0)
+		(effects
+			(font
+				(size 1.27 1.27)
+			)
 		)
 	)
@@
 		)
 	)
-	(text "Fucked up pinout"
+	(text "Wrong pinout of U106"
 		(exclude_from_sim no)
-		(at 139.7 172.466 0)
+		(at 143.51 171.958 0)
 		(effects
 			(font
@@
 		)
 	)
-	(text "changed 6.8u to 10u\n"
+	(text "C150, C153 - 10u"
 		(exclude_from_sim no)
 		(at 166.878 39.116 0)
