File: Differential_Probe_PCB/Differential_Probe.kicad_sch (KiCad schematic)
At the start: 11 parts, among them J101 Conn_01x01_Socket, J102 Conn_Coaxial, J103 Conn_01x01_Socket, SW101 SW_SPDT, SW102 SW_SPDT

Commit message: .
Parts:
- removed D101, D102, D113: BLED, Diode_SMD:D_1206_3216Metric, symbol Device:LED
- removed R101, R102, R154: 1k, Resistor_SMD:R_0603_1608Metric, symbol Device:R_Small
- removed SW101: SW_SPDT, SamacSys_Parts:MHPS2285, symbol Switch:SW_SPDT
- removed SW102: SW_SPDT, SamacSys_Parts:MHPS2285, symbol Switch:SW_Push
- J102: footprint Connector_Coaxial:BNC_Amphenol_031-6575_Horizontal -> SamacSys_Parts:2269901
Connections:
- no-connect marks 1 -> 0
Other:
- added sheet Buttons_indication (Buttons_indication.kicad_sch)
- sheet Amplifier ports: added Single_ended_input; removed none

Commit message: After 1st debug update to sch
Other:
- note added: "all 100n 0603 changed to 150n 0603"
Changed lines of the file:
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@@
+		)
+	)
+	(text "all 100n 0603 changed to 150n 0603\n"
+		(exclude_from_sim no)
+		(at 148.082 164.592 0)
+		(effects
+			(font
+				(size 1.27 1.27)
+				(color 255 0 0 1)
+			)
 		)
 	)

Commit message: .
Changed lines of the file:
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@@
 	(text "all 100n 0603 changed to 150n 0603\n"
 		(exclude_from_sim no)
-		(at 148.082 164.592 0)
+		(at 109.982 187.96 0)
 		(effects
 			(font
