File: Differential_Probe_PCB/Power_supply.kicad_sch (KiCad schematic)
At the start: 45 parts, among them J104 USB_C_Receptacle_PowerOnly_6P, U101 TPS7A39, U102 TPS65130RGE

Commit message: .
Parts:
- added TP108, TP109, TP110, TP111: TestPoint, TestPoint:TestPoint_THTPad_D1.0mm_Drill0.5mm, symbol Connector:TestPoint
- C139: value xxx -> 6.8p
- C142: value 220n -> 6.8p
- C146: value xxx -> 10n
- C147: value xxx -> 4.7n
- J104: footprint Connector_USB:USB_C_Receptacle_HRO_TYPE-C-31-M-17 -> Connector_USB:USB_C_Receptacle_GCT_USB4125-xx-x_6P_TopMnt_Horizontal
- R130: value 90.9k -> 100k
- R131: value xxx -> 1M
- R132: value xxx -> 88k
- R133: value xxx -> 100k
- R135: value xxx -> 1.3M
Connections:
- net +12V: now also TP110.1
- net +15V: now also TP108.1
- net -12V: now also TP111.1
- net -15V: now also TP109.1
Other:
- moved on the sheet: C142, R135

Commit message: After 1st debug update to sch
Parts:
- R130: value 100k -> 90.9k
Other:
- note added: "FB103&FB104 - 0R"
- note added: "R130- 10k R129- 1k C133 DNP"
- note added: "R134 -> 150R"
Changed lines of the file:
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@@
 	(generator_version "9.0")
 	(paper "A4")
+	(text "R130- 10k\nR129- 1k\nC133 DNP\n"
+		(exclude_from_sim no)
+		(at 208.534 63.5 0)
+		(effects
+			(font
+				(size 1.27 1.27)
+				(color 255 0 0 1)
+			)
+		)
+	)
+	(text "R134 -> 150R\n"
+		(exclude_from_sim no)
+		(at 164.592 142.24 0)
+		(effects
+			(font
+				(size 1.27 1.27)
+				(color 255 0 0 1)
+			)
+		)
+	)
+	(text "FB103&FB104 - 0R"
+		(exclude_from_sim no)
+		(at 128.016 49.53 0)
+		(effects
+			(font
+				(size 1.27 1.27)
+				(color 255 0 0 1)
+			)
+		)
+	)
 	(junction
 		(at 241.554 129.032)
@@
 			)
 		)
-		(property "Value" "100k"
+		(property "Value" "90.9k"
 			(at 212.09 53.8479 0)
 			(effects
